Commit message: More updates to Gears description, work on diff suspension plugin. Unfortunately, it works, but it doesn't keep the chassis steady.

File: testrover_description/urdf/gears_smp.urdf.xacro (robot description, xacro)
@@ -4,10 +4,4 @@
     A rough model of the Gears SMP rover. Details at http://www.gearseds.com/surface_mobility_platform.html
 -->
-    <!-- Load the Gazebo-ROS Control interface -->
-    <gazebo>
-        <plugin name="gazebo_ros_control" filename="libgazebo_ros_control.so">
-            <!--<robotNamespace></robotNamespace>-->
-        </plugin>
-    </gazebo>
     <!-- Add relevant macros -->
     <xacro:include filename="$(find testrover_description)/urdf/macros/components/wheel.urdf.xacro" />
@@ -19,10 +13,10 @@
     <xacro:property name="chassis_width" value=".14"/>
     <xacro:property name="chassis_height" value=".0889"/>
-    <xacro:property name="chassis_mass" value="5.0"/>
+    <xacro:property name="chassis_mass" value="1.584994"/>
     <!-- Rocker dimensions and positioning -->
     <xacro:property name="rocker_length" value=".2667"/>
     <xacro:property name="rocker_width" value=".03175"/>
     <xacro:property name="rocker_height" value=".03175"/>
-    <xacro:property name="rocker_mass" value="0.5"/>
+    <xacro:property name="rocker_mass" value="1.387336"/>
     <xacro:property name="rocker_x" value="0.0"/>
     <xacro:property name="rocker_y" value="${0.12065-0.5*rocker_width}"/>
@@ -31,5 +25,5 @@
     <xacro:property name="wheel_radius" value="0.08255"/>
     <xacro:property name="wheel_depth" value=".0508"/>
-    <xacro:property name="wheel_mass" value="1.5"/>
+    <xacro:property name="wheel_mass" value="0.283642"/>
     <!-- Wheel positioning -->
     <xacro:property name="wheel_spacing_x" value="0.19678256"/>
@@ -53,13 +47,15 @@
             <origin xyz="0 0 0" rpy="0 0 0"/>
             <mass value="${chassis_mass}"/>
-            <inertia ixx="1.25" ixy="0.0" ixz="0.0"
-                     iyy="7.0" iyz="0.0" izz="8.0" />
-        </inertial>
+            <inertia
+                ixx="0.01042" ixy="0.001177" ixz="-0.0008871"
+                iyy="0.01045" iyz="0.0002226"
+                izz="0.01817"/>
+            </inertial>
     </link>
     <!-- Add the rockers -->
-    <xacro:rocker prefix="left" parent="base_link" rockerx="${rocker_length}" rockery="${rocker_width}" rockerz="${rocker_height}" rockerkg="${rocker_mass}">
+    <xacro:rocker prefix="left" parent="base_link" rockerx="${rocker_length}" rockery="${rocker_width}" rockerz="${rocker_height}" rockerkg="${rocker_mass}" mimicing="0" mimic_joint="">
         <origin xyz="${rocker_x} ${rocker_y} ${-rocker_z}" rpy="0 0 0"/>
     </xacro:rocker>
-    <xacro:rocker prefix="right" parent="base_link" rockerx="${rocker_length}" rockery="${rocker_width}" rockerz="${rocker_height}" rockerkg="${rocker_mass}">
+    <xacro:rocker prefix="right" parent="base_link" rockerx="${rocker_length}" rockery="${rocker_width}" rockerz="${rocker_height}" rockerkg="${rocker_mass}"  mimicing="1" mimic_joint="left_rocker_joint">
         <origin xyz="${rocker_x} ${-rocker_y} ${-rocker_z}" rpy="0 0 0"/>
     </xacro:rocker>
@@ -77,3 +73,17 @@
         <origin xyz="${-wheel_spacing_x} ${-wheel_spacing_y} ${wheel_spacing_z}" rpy="0 0 0"/>
     </xacro:wheel>
+    <!-- Add the differential suspenion sim plugin and reference the two rockers, as well as the force constant between them -->
+    <gazebo>
+        <plugin name="rover_gazebo_diff_plugin" filename="librover_gazebo_diff_plugin.so">
+            <jointA>left_rocker_joint</jointA>
+            <jointB>right_rocker_joint</jointB>
+            <forceConstant>100.0</forceConstant>
+        </plugin>
+    </gazebo>
+        <!-- Load the Gazebo-ROS Control interface -->
+    <gazebo>
+        <plugin name="gazebo_ros_control" filename="libgazebo_ros_control.so">
+            <!--<robotNamespace></robotNamespace>-->
+        </plugin>
+    </gazebo>
 </robot>

File: testrover_description/urdf/macros/components/rocker.urdf.xacro (robot description, xacro)
@@ -3,5 +3,5 @@
 <robot xmlns:xacro="http://www.ros.org/wiki/xacro">
 <!-- Description for a simple rocker bar. Could also be used as a bogie? -->
-<xacro:macro name="rocker" params="prefix parent rockerx rockery rockerz rockerkg *origin">
+<xacro:macro name="rocker" params="prefix parent rockerx rockery rockerz rockerkg mimicing mimic_joint *origin">
     <!-- Create a link for the wheels -->
     <link name="${prefix}_rocker_link">
@@ -23,9 +23,11 @@
             <origin xyz="0 0 0" rpy="0 0 0"/>
             <mass value="${rockerkg}"/>
-            <inertia ixx="0.001" ixy="0" ixz="0"
-                        iyy="0.001" iyz="0" izz="0.001" />
+            <inertia
+                ixx="0.002956" ixy="-0.000001489324" ixz="-0.000008103407"
+                iyy="0.02924"  iyz="0.00007112"
+                izz="0.02832"/>
         </inertial>
     </link>
-    <joint name="${prefix}_rocker_joint" type="continuous">
+    <joint name="${prefix}_rocker_joint" type="revolute">
         <parent link="${parent}"/>
         <child link="${prefix}_rocker_link"/>
@@ -36,4 +38,9 @@
         <!-- Specify rotation axis of wheel -->
         <axis xyz="0 1 0"/>
+        <limit effort="100.0" lower="-0.24" upper="0.24" velocity="100.0"/>
+        <!-- Set joint to mimic another joint specified above if true -->
+        <xacro:if value="${mimicing == 1}">
+        <mimic joint= "${mimic_joint}"/>
+        </xacro:if>
     </joint>
 </xacro:macro>

File: testrover_description/urdf/macros/components/wheel.urdf.xacro (robot description, xacro)
@@ -23,6 +23,8 @@
             <origin xyz="0 0 0" rpy="0 0 0"/>
             <mass value="${wheelkg}"/>
-            <inertia ixx="0.08" ixy="0" ixz="0"
-                        iyy="0.14" iyz="0" izz="0.08" />
+            <inertia
+                ixx="0.000391"  ixy="0.00000123962" ixz="5.52582e-7"
+                iyy="0.0004716" iyz="-0.000002082042"
+                izz="0.000391"/>
         </inertial>
     </link>
