Commit message: Added Gears SMP description and work on differential suspension sim plugin.

File: testrover_description/urdf/macros/components/wheel.urdf.xacro (robot description, xacro)
@@ -1,7 +1,7 @@
 <?xml version="1.0"?>
-<!-- define xacro as the namespace referencing the xacro format. Important for compiling Xacro files and macros-->
+<!-- define xacro as the namespace referencing the xacro format. Important for compiling xacro files and macros-->
 <robot xmlns:xacro="http://www.ros.org/wiki/xacro">
-<!-- Macro detailing the reactions of each wheel -->
-<xacro:macro name="wheel" params="prefix parent *origin">
+<!-- Macro detailing the details of each wheel -->
+<xacro:macro name="wheel" params="prefix parent wheelrad wheeldepth wheelkg *origin">
     <!-- Create a link for the wheels -->
     <link name="${prefix}_wheel_link">
@@ -10,5 +10,5 @@
             <origin xyz="0 0 0" rpy="${PI/2} 0 0"/>
             <geometry>
-                <cylinder radius="${wheel_radius}" length="${wheel_depth}"/>
+                <cylinder radius="${wheelrad}" length="${wheeldepth}"/>
             </geometry>
         </visual>
@@ -16,5 +16,5 @@
             <origin xyz="0 0 0" rpy="${PI/2} 0 0"/>
             <geometry>
-                <cylinder radius="${wheel_radius}" length="${wheel_depth}"/>
+                <cylinder radius="${wheelrad}" length="${wheeldepth}"/>
             </geometry>
         </collision>
@@ -22,5 +22,5 @@
         <inertial>
             <origin xyz="0 0 0" rpy="0 0 0"/>
-            <mass value="0.477"/>
+            <mass value="${wheelkg}"/>
             <inertia ixx="0.08" ixy="0" ixz="0"
                         iyy="0.14" iyz="0" izz="0.08" />
@@ -31,6 +31,5 @@
         <child link="${prefix}_wheel_link"/>
         <!--
-            Use insert_block to specify joint (and wheel) position in wheel
-            declaration later
+            Use insert_block to specify joint (and wheel) position in wheel declaration
         -->
         <xacro:insert_block name="origin"/>

File: testrover_description/urdf/testrover.urdf.xacro (robot description, xacro)
@@ -12,5 +12,5 @@
     <gazebo>
         <plugin name="gazebo_ros_control" filename="libgazebo_ros_control.so">
-            <!--<robotNamespace>/testrover</robotNamespace>-->
+            <!--<robotNamespace></robotNamespace>-->
         </plugin>
     </gazebo>
@@ -60,17 +60,18 @@
     </link>
     <!-- Declare the wheels and their origins -->
-    <xacro:wheel prefix="front_left" parent="base_link">
+    <xacro:wheel prefix="front_left" parent="base_link" wheelrad="${wheel_radius}" wheeldepth="${wheel_depth}" wheelkg="${wheel_mass}" >
         <origin xyz="${wheel_spacing_x} ${wheel_spacing_y} 0.0" rpy="0 0 0"/>
     </xacro:wheel>
-    <xacro:wheel prefix="rear_left" parent="base_link">
+    <xacro:wheel prefix="rear_left" parent="base_link" wheelrad="${wheel_radius}" wheeldepth="${wheel_depth}" wheelkg="${wheel_mass}">
         <origin xyz="${-wheel_spacing_x} ${wheel_spacing_y} 0.0" rpy="0 0 0"/>
     </xacro:wheel>
-    <xacro:wheel prefix="front_right" parent="base_link">
+    <xacro:wheel prefix="front_right" parent="base_link" wheelrad="${wheel_radius}" wheeldepth="${wheel_depth}" wheelkg="${wheel_mass}">
         <origin xyz="${wheel_spacing_x} ${-wheel_spacing_y} 0.0" rpy="0 0 0"/>
     </xacro:wheel>
-    <xacro:wheel prefix="rear_right" parent="base_link">
+    <xacro:wheel prefix="rear_right" parent="base_link" wheelrad="${wheel_radius}" wheeldepth="${wheel_depth}" wheelkg="${wheel_mass}">
         <origin xyz="${-wheel_spacing_x} ${-wheel_spacing_y} 0.0" rpy="0 0 0"/>
     </xacro:wheel>
-    <xacro:kinect parent="base_link">\
+    <!-- Add the kinect at its origin -->
+    <xacro:kinect parent="base_link">
         <origin xyz="${camera_mnt_x} ${camera_mnt_y} ${camera_mnt_z}" rpy="0 0 0"/>
     </xacro:kinect>
