Commit message: Reorganized file layout

File: rover_robots/gears_smp/urdf/gears_smp.urdf.xacro (robot description, xacro)
@@ -5,6 +5,6 @@
 -->
     <!-- Add relevant macros -->
-    <xacro:include filename="$(find testrover_description)/urdf/macros/components/wheel.urdf.xacro" />
-    <xacro:include filename="$(find testrover_description)/urdf/macros/components/rocker.urdf.xacro" />
+    <xacro:include filename="$(find rover_robots)/urdf/macros/components/wheel.urdf.xacro" />
+    <xacro:include filename="$(find rover_robots)/urdf/macros/components/rocker.urdf.xacro" />
     <xacro:property name="PI" value="3.1415926535897931" />
     <!-- All dimensions in SI units (kg, m, etc.)-->
@@ -56,20 +56,44 @@
     <xacro:rocker prefix="left" parent="base_link" rockerx="${rocker_length}" rockery="${rocker_width}" rockerz="${rocker_height}" rockerkg="${rocker_mass}" mimicing="0" mimic_joint="">
         <origin xyz="${rocker_x} ${rocker_y} ${-rocker_z}" rpy="0 0 0"/>
+        <inertia
+            ixx="0.002956" ixy="-0.000001489324" ixz="-0.000008103407"
+            iyy="0.02924"  iyz="0.00007112"
+            izz="0.02832"/>
     </xacro:rocker>
     <xacro:rocker prefix="right" parent="base_link" rockerx="${rocker_length}" rockery="${rocker_width}" rockerz="${rocker_height}" rockerkg="${rocker_mass}"  mimicing="1" mimic_joint="left_rocker_joint">
         <origin xyz="${rocker_x} ${-rocker_y} ${-rocker_z}" rpy="0 0 0"/>
+        <inertia
+            ixx="0.002956" ixy="-0.000001489324" ixz="-0.000008103407"
+            iyy="0.02924"  iyz="0.00007112"
+            izz="0.02832"/>
     </xacro:rocker>
-    <!-- Declare the wheels and their origins -->
+    <!-- Add the wheels -->
     <xacro:wheel prefix="front_left" parent="left_rocker_link" wheelrad="${wheel_radius}" wheeldepth="${wheel_depth}" wheelkg="${wheel_mass}" >
         <origin xyz="${wheel_spacing_x} ${wheel_spacing_y} ${wheel_spacing_z}" rpy="0 0 0"/>
+        <inertia
+            ixx="0.000391"  ixy="0.00000123962" ixz="5.52582e-7"
+            iyy="0.0004716" iyz="-0.000002082042"
+            izz="0.000391"/>
     </xacro:wheel>
     <xacro:wheel prefix="rear_left" parent="left_rocker_link" wheelrad="${wheel_radius}" wheeldepth="${wheel_depth}" wheelkg="${wheel_mass}">
         <origin xyz="${-wheel_spacing_x} ${wheel_spacing_y} ${wheel_spacing_z}" rpy="0 0 0"/>
+        <inertia
+            ixx="0.000391"  ixy="0.00000123962" ixz="5.52582e-7"
+            iyy="0.0004716" iyz="-0.000002082042"
+            izz="0.000391"/>
     </xacro:wheel>
     <xacro:wheel prefix="front_right" parent="right_rocker_link" wheelrad="${wheel_radius}" wheeldepth="${wheel_depth}" wheelkg="${wheel_mass}">
         <origin xyz="${wheel_spacing_x} ${-wheel_spacing_y} ${wheel_spacing_z}" rpy="0 0 0"/>
+        <inertia
+            ixx="0.000391"  ixy="0.00000123962" ixz="5.52582e-7"
+            iyy="0.0004716" iyz="-0.000002082042"
+            izz="0.000391"/>
     </xacro:wheel>
     <xacro:wheel prefix="rear_right" parent="right_rocker_link" wheelrad="${wheel_radius}" wheeldepth="${wheel_depth}" wheelkg="${wheel_mass}">
         <origin xyz="${-wheel_spacing_x} ${-wheel_spacing_y} ${wheel_spacing_z}" rpy="0 0 0"/>
+        <inertia
+            ixx="0.000391"  ixy="0.00000123962" ixz="5.52582e-7"
+            iyy="0.0004716" iyz="-0.000002082042"
+            izz="0.000391"/>
     </xacro:wheel>
     <!-- Add the differential suspenion sim plugin and reference the two rockers, as well as the force constant between them -->

File: rover_robots/testrover/urdf/testrover.urdf.xacro (robot description, xacro)
@@ -16,7 +16,7 @@
     </gazebo>
     <!-- Define the kinect -->
-    <xacro:include filename="$(find testrover_description)/urdf/macros/accessories/kinect.urdf.xacro" />
+    <xacro:include filename="$(find rover_robots)/urdf/macros/accessories/kinect.urdf.xacro" />
     <!-- Macro detailing the reactions of each wheel -->
-    <xacro:include filename="$(find testrover_description)/urdf/macros/components/wheel.urdf.xacro" />
+    <xacro:include filename="$(find rover_robots)/urdf/macros/components/wheel.urdf.xacro" />
     <xacro:property name="PI" value="3.1415926535897931" />
     <!-- All dimensions in SI units (kg, m, etc.)-->
@@ -62,13 +62,21 @@
     <xacro:wheel prefix="front_left" parent="base_link" wheelrad="${wheel_radius}" wheeldepth="${wheel_depth}" wheelkg="${wheel_mass}" >
         <origin xyz="${wheel_spacing_x} ${wheel_spacing_y} 0.0" rpy="0 0 0"/>
+        <inertia ixx="0.08" ixy="0" ixz="0"
+                 iyy="0.14" iyz="0" izz="0.08" />
     </xacro:wheel>
     <xacro:wheel prefix="rear_left" parent="base_link" wheelrad="${wheel_radius}" wheeldepth="${wheel_depth}" wheelkg="${wheel_mass}">
         <origin xyz="${-wheel_spacing_x} ${wheel_spacing_y} 0.0" rpy="0 0 0"/>
+        <inertia ixx="0.08" ixy="0" ixz="0"
+                 iyy="0.14" iyz="0" izz="0.08" />
     </xacro:wheel>
     <xacro:wheel prefix="front_right" parent="base_link" wheelrad="${wheel_radius}" wheeldepth="${wheel_depth}" wheelkg="${wheel_mass}">
         <origin xyz="${wheel_spacing_x} ${-wheel_spacing_y} 0.0" rpy="0 0 0"/>
+        <inertia ixx="0.08" ixy="0" ixz="0"
+                 iyy="0.14" iyz="0" izz="0.08" />
     </xacro:wheel>
     <xacro:wheel prefix="rear_right" parent="base_link" wheelrad="${wheel_radius}" wheeldepth="${wheel_depth}" wheelkg="${wheel_mass}">
         <origin xyz="${-wheel_spacing_x} ${-wheel_spacing_y} 0.0" rpy="0 0 0"/>
+        <inertia ixx="0.08" ixy="0" ixz="0"
+                 iyy="0.14" iyz="0" izz="0.08" />
     </xacro:wheel>
     <!-- Add the kinect at its origin -->

File: rover_robots/urdf/macros/components/rocker.urdf.xacro (robot description, xacro)
@@ -3,5 +3,5 @@
 <robot xmlns:xacro="http://www.ros.org/wiki/xacro">
 <!-- Description for a simple rocker bar. Could also be used as a bogie? -->
-<xacro:macro name="rocker" params="prefix parent rockerx rockery rockerz rockerkg mimicing mimic_joint *origin">
+<xacro:macro name="rocker" params="prefix parent rockerx rockery rockerz rockerkg mimicing mimic_joint *origin *inertia">
     <!-- Create a link for the wheels -->
     <link name="${prefix}_rocker_link">
@@ -23,4 +23,5 @@
             <origin xyz="0 0 0" rpy="0 0 0"/>
             <mass value="${rockerkg}"/>
+            <xacro:insert_block name="inertia"/>
             <inertia
                 ixx="0.002956" ixy="-0.000001489324" ixz="-0.000008103407"

File: rover_robots/urdf/macros/components/wheel.urdf.xacro (robot description, xacro)
@@ -3,5 +3,5 @@
 <robot xmlns:xacro="http://www.ros.org/wiki/xacro">
 <!-- Macro detailing the details of each wheel -->
-<xacro:macro name="wheel" params="prefix parent wheelrad wheeldepth wheelkg *origin">
+<xacro:macro name="wheel" params="prefix parent wheelrad wheeldepth wheelkg *origin *inertia">
     <!-- Create a link for the wheels -->
     <link name="${prefix}_wheel_link">
@@ -23,8 +23,5 @@
             <origin xyz="0 0 0" rpy="0 0 0"/>
             <mass value="${wheelkg}"/>
-            <inertia
-                ixx="0.000391"  ixy="0.00000123962" ixz="5.52582e-7"
-                iyy="0.0004716" iyz="-0.000002082042"
-                izz="0.000391"/>
+            <xacro:insert_block name="inertia"/>
         </inertial>
     </link>
